File: hardware/pidplate-mk-2.brd (EAGLE design)
At the start: 49 x 59 mm, 45 parts, among them J1 M06X2PTH, Q1 2N7000, Q2 2N3904, U1 ATMEGA328P, U3 VSK-S1, Y1 16MHz

Commit message: misc changes upon receiving boards, and some work maybe on the firmware
Parts:
- removed AC(L), AC(N): M01PTH-1.2MM, A_butts:1X01-1.2MM
- added AVRISP: AVR_SPI_PRG_6PTH, A_butts:2X3
- added C10: 0.1uF, A_butts:C025-024X044
- added DIAG, RELAY: LED3MM, A_butts:LED3MM
- added JP1: M023.5MM, A_butts:SCREWTERMINAL-3.5MM-2
- added R5, R7: 330R, A_butts:RESISTOR-AXIAL-PTH-5.08MM
- moved R4 59.7 mm to (62.3, 23.0), turned to 0 degrees
- moved PWR 56.2 mm to (54.5, 23.5), turned to 0 degrees
- moved H5 23.0 mm to (62.5, 40.0)
- moved H1 16.8 mm to (61.5, 42.0)
- moved PTC 7.78 mm to (4.50, 41.9), turned to 270 degrees
- moved CX1 7.52 mm to (42.5, 54.0)
- moved MOV1 2.24 mm to (45.0, 45.5), turned to 180 degrees
Connections:
- removed net N$11: AC(N).P$1, CX1.2, MOV1.1, U3.AC2
- removed net N$12: AC(L).P$1, CX1.1, MOV1.2, U3.AC1
- new net AC(L): CX1.1, JP1.2, MOV1.2, U3.AC1
- new net AC(N): CX1.2, JP1.1, MOV1.1, U3.AC2
- new net DIAG: R5.P$2, U1.11
- new net N$13: R7.P$1, RELAY.A
- new net N$14: C10.2, FTDI.1
- new net N$2: DIAG.A, R5.P$1
- net DB7: now also AVRISP.4
- net GND: now also AVRISP.6, DIAG.K
- net N$9: now also RELAY.K
- net RESET: now also AVRISP.5, C10.1; no longer FTDI.1
- net RS: now also AVRISP.1
- net RW: now also AVRISP.3
- net RX: now also FTDI.3; no longer FTDI.2
- net TX: now also FTDI.2; no longer FTDI.3
- net VCC: now also AVRISP.2, R7.P$2
Routing:
- net RESET: track 86.6 -> 69.2 mm
- net N$11: track 15.0 -> 0.00 mm
- net N$12: track 13.4 -> 0.00 mm
- net VCC: track 95.2 -> 102.1 mm
- net N$1: track 16.6 -> 21.7 mm
- net N$10: track 3.00 -> 0.00 mm
- net RX: track 52.4 -> 53.5 mm
Other:
- outline, holes or cut-outs redrawn
