File: hardware/pidplate-mk-2.sch (EAGLE design)
At the start: 41 parts, among them J1 M06X2PTH, Q1 2N7000, Q2 2N3904, U1 ATMEGA328P, U3 VSK-S1, Y1 16MHz

Commit message: misc changes upon receiving boards, and some work maybe on the firmware
Parts:
- removed AC(L), AC(N): M01PTH-1.2MM, A_butts:M01PTH-1.2MM
- added AVRISP: AVR_SPI_PRG_6PTH, A_butts:AVR_SPI_PRG_6PTH
- added C10: 0.1uF, A_butts:CAPACITOR-CERAMIC025-024X044
- added DIAG, RELAY: LED3MM, A_butts:LED3MM
- added JP1: M023.5MM, A_butts:M023.5MM
- added R5, R7: 330R, A_butts:RESISTORPTH-AXIAL-5.08MM
Connections:
- removed net N$11: AC(N).1, CX1.2, MOV1.P$1, U3.AC(N)
- removed net N$12: AC(L).1, CX1.1, MOV1.P$2, U3.AC(L)
- new net AC(L): CX1.1, JP1.2, MOV1.P$2, U3.AC(L)
- new net AC(N): CX1.2, JP1.1, MOV1.P$1, U3.AC(N)
- new net DIAG: R5.2, U1.PD5(T1)
- new net N$13: R7.1, RELAY.A
- new net N$14: C10.2, FTDI.1
- new net N$2: DIAG.A, R5.1
- net DB7: now also AVRISP.4
- net GND: now also AVRISP.6, DIAG.C
- net N$9: now also RELAY.C
- net RESET: now also AVRISP.5, C10.1; no longer FTDI.1
- net RS: now also AVRISP.1
- net RW: now also AVRISP.3
- net RX: now also FTDI.3; no longer FTDI.2
- net TX: now also FTDI.2; no longer FTDI.3
- net VCC: now also AVRISP.2, R7.2
Other:
- moved on the sheet: R3, RESET, SSR
