File: hardware/pidshield-mk-1.sch (EAGLE design)
At the start: 32 parts, among them IC1 MAX31855, IC2 LM2931-3.3V, Q1 2N7000, Q2 2N7000, Q3 2N7000, Q4 2N7000, U1 ARDUINO_SHIELDINSIDER

Commit message: think i've got the layout how i want it
Parts:
- removed IC2: LM2931-3.3V, A_butts:V_REG_78XXTO-92-INLINE
- removed SJ1: JUMPER-PAD-2-NC_BY_TRACE, A_butts:JUMPER-PAD-2-NC_BY_TRACE
- C1, C2: value 0.1uF -> 1uF
- C3: value 0.1uF -> 0.01uF
- C4, C5: value 1uF -> 0.1uF
- Q2, Q3, Q4: device A_butts:MOSFET-NCHANNEL2N7000 -> A_butts:MOSFET-NCHANNEL2N7000-AMMO
- TC1: value THERMOCOUPLE-CONNECTORMINI-PCB -> PCC-SMP-K
Connections:
- removed net N$1: SJ1.2, U1.3.3V
- net 3.3V: now also U1.3.3V; no longer IC2.OUT, SJ1.1
- net 5V: now also C1.2; no longer C1.1, IC2.IN
- net GND: now also C1.1, R9.1, RESET.1; no longer C1.2, IC2.GND, R9.2, RESET.2
- net RESET: now also RESET.2; no longer RESET.1
- net SSR: now also R9.2; no longer R9.1
Other:
- note removed: "(Optional) 3.3 Voltage Regulator For hosts lacking a 3.3V supply"
- note removed: "(Optional) Normally connected trace jumper. Cut if you don't want to use the host's 3.3V line (e.g., if it's not actually 3.3V)"
- moved on the sheet: C1, C2, C3, C4, C5, LCD, LED1, Q1, R10, R11, R7, R8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
