File: hardware/pidshield-mk-2.brd (EAGLE design)
At the start: 52 x 37.5 mm, 28 parts, among them IC1 MAX31855, Q1 2N7000

Commit message: in progress commit
Routing:
- net 3.3V: track 0.00 -> 79.3 mm
- net RESET: track 0.00 -> 47.7 mm, vias 0 -> 2
- net MISO: track 0.00 -> 37.5 mm, vias 0 -> 1
- net SCK: track 0.00 -> 37.1 mm
- net CS: track 0.00 -> 29.1 mm
- net SCL: track 0.00 -> 21.7 mm
- net SDA: track 0.00 -> 18.3 mm
- net N$2: track 0.00 -> 14.4 mm
- net SSR: track 0.00 -> 13.9 mm
- net N$3: track 0.00 -> 11.2 mm
- net N$4: track 0.00 -> 10.6 mm
- net YELLOW(+): track 0.00 -> 10.1 mm
- net RED(-): track 0.00 -> 10.1 mm
- net MOSI: track 0.00 -> 6.66 mm
- net GND: track 3.00 -> 3.50 mm
