File: hardware/ir-sensor-breakout-mk-2.0.sch (EAGLE design)
At the start: 6 parts, among them U1 MLX906145V-PTH

Commit message: fiddling with the pth breakout
Parts:
- added H1, H2, H3, H4: HOLE#2, A_butts:HOLE#2
- R1, R2: device A_butts:RESISTORPTH-AXIAL-7.62MM -> A_butts:RESISTORPTH-AXIAL-5.08MM
Connections:
- net GND: now also I2C.1; no longer I2C.4
- net SCL: now also I2C.4; no longer I2C.1
- net SDA: now also I2C.3; no longer I2C.2
- net VCC: now also I2C.2; no longer I2C.3
Other:
- moved on the sheet: I2C
Changed lines of the file:
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@@
 <part name="U1" library="A_butts" deviceset="MLX90614" device="5V-PTH"/>
 <part name="C1" library="A_butts" deviceset="CAPACITOR-CERAMIC" device="025-024X044" value="100nF"/>
-<part name="R1" library="A_butts" deviceset="RESISTOR" device="PTH-AXIAL-7.62MM" value="10k"/>
-<part name="R2" library="A_butts" deviceset="RESISTOR" device="PTH-AXIAL-7.62MM" value="10k"/>
+<part name="R1" library="A_butts" deviceset="RESISTOR" device="PTH-AXIAL-5.08MM" value="10k"/>
+<part name="R2" library="A_butts" deviceset="RESISTOR" device="PTH-AXIAL-5.08MM" value="10k"/>
 <part name="SUPPLY2" library="A_butts" deviceset="VCC" device=""/>
 <part name="GND2" library="A_butts" deviceset="GND" device=""/>
 <part name="SUPPLY3" library="A_butts" deviceset="VCC" device=""/>
 <part name="SUPPLY4" library="A_butts" deviceset="VCC" device=""/>
-<part name="GND4" library="A_butts" deviceset="GND" device=""/>
-<part name="SUPPLY6" library="A_butts" deviceset="VCC" device=""/>
+<part name="H1" library="A_butts" deviceset="HOLE" device="#2"/>
+<part name="H2" library="A_butts" deviceset="HOLE" device="#2"/>
+<part name="H3" library="A_butts" deviceset="HOLE" device="#2"/>
+<part name="H4" library="A_butts" deviceset="HOLE" device="#2"/>
+<part name="GND3" library="A_butts" deviceset="GND" device=""/>
+<part name="SUPPLY5" library="A_butts" deviceset="VCC" device=""/>
 </parts>
 <sheets>
@@
 <instance part="SUPPLY1" gate="G$1" x="76.2" y="83.82"/>
 <instance part="GND1" gate="1" x="76.2" y="60.96"/>
-<instance part="I2C" gate="G$1" x="38.1" y="66.04" rot="MR180"/>
+<instance part="I2C" gate="G$1" x="40.64" y="63.5"/>
 <instance part="U1" gate="G$1" x="88.9" y="73.66"/>
 <instance part="C1" gate="G$1" x="114.3" y="43.18"/>
@@
 <instance part="SUPPLY3" gate="G$1" x="124.46" y="50.8"/>
 <instance part="SUPPLY4" gate="G$1" x="134.62" y="50.8"/>
-<instance part="GND4" gate="1" x="55.88" y="55.88"/>
-<instance part="SUPPLY6" gate="G$1" x="55.88" y="66.04"/>
+<instance part="H1" gate="G$1" x="5.08" y="180.34"/>
+<instance part="H2" gate="G$1" x="243.84" y="180.34"/>
+<instance part="H3" gate="G$1" x="243.84" y="33.02"/>
+<instance part="H4" gate="G$1" x="5.08" y="5.08"/>
+<instance part="GND3" gate="1" x="58.42" y="55.88"/>
+<instance part="SUPPLY5" gate="G$1" x="58.42" y="66.04"/>
 </instances>
 <busses>
@@
 </segment>
 <segment>
-<wire x1="43.18" y1="63.5" x2="55.88" y2="63.5" width="0.1524" layer="91"/>
-<pinref part="SUPPLY6" gate="G$1" pin="VCC"/>
-<wire x1="55.88" y1="63.5" x2="55.88" y2="66.04" width="0.1524" layer="91"/>
-<pinref part="I2C" gate="G$1" pin="3"/>
+<wire x1="45.72" y1="63.5" x2="58.42" y2="63.5" width="0.1524" layer="91"/>
+<pinref part="SUPPLY5" gate="G$1" pin="VCC"/>
+<wire x1="58.42" y1="63.5" x2="58.42" y2="66.04" width="0.1524" layer="91"/>
+<pinref part="I2C" gate="G$1" pin="2"/>
 </segment>
 </net>
@@
 </segment>
 <segment>
-<pinref part="GND4" gate="1" pin="GND"/>
-<wire x1="43.18" y1="60.96" x2="55.88" y2="60.96" width="0.1524" layer="91"/>
-<wire x1="55.88" y1="60.96" x2="55.88" y2="58.42" width="0.1524" layer="91"/>
-<pinref part="I2C" gate="G$1" pin="4"/>
+<pinref part="GND3" gate="1" pin="GND"/>
+<wire x1="45.72" y1="60.96" x2="58.42" y2="60.96" width="0.1524" layer="91"/>
+<wire x1="58.42" y1="60.96" x2="58.42" y2="58.42" width="0.1524" layer="91"/>
+<pinref part="I2C" gate="G$1" pin="1"/>
 </segment>
 </net>
@@
 </segment>
 <segment>
-<wire x1="45.72" y1="66.04" x2="43.18" y2="66.04" width="0.1524" layer="91"/>
-<label x="45.72" y="66.04" size="1.27" layer="95" xref="yes"/>
-<pinref part="I2C" gate="G$1" pin="2"/>
+<wire x1="48.26" y1="66.04" x2="45.72" y2="66.04" width="0.1524" layer="91"/>
+<label x="48.26" y="66.04" size="1.27" layer="95" xref="yes"/>
+<pinref part="I2C" gate="G$1" pin="3"/>
 </segment>
 </net>
@@
 </segment>
 <segment>
-<wire x1="45.72" y1="68.58" x2="43.18" y2="68.58" width="0.1524" layer="91"/>
-<label x="45.72" y="68.58" size="1.27" layer="95" xref="yes"/>
-<pinref part="I2C" gate="G$1" pin="1"/>
+<wire x1="48.26" y1="68.58" x2="45.72" y2="68.58" width="0.1524" layer="91"/>
+<label x="48.26" y="68.58" size="1.27" layer="95" xref="yes"/>
+<pinref part="I2C" gate="G$1" pin="4"/>
 </segment>
 </net>
